File: Drone_FCU_rev1.kicad_sch (KiCad schematic)
At the start: 31 parts, among them J1 Conn_01x02_Pin, P1 USB_C_Plug_USB2.0, SW1 SW_Push, U1 STM32F722VETx, Y2 16MHz

Commit message: Update flight controller schematic and libraries
Parts:
- removed C10, C9: 1u, symbol Device:C
- removed C7: 10u, symbol Device:C
- removed C8: 100n, symbol Device:C
- removed FB1: 120R, symbol Device:FerriteBead
- removed P1: USB_C_Plug_USB2.0, symbol Connector:USB_C_Plug_USB2.0
- added C16: 10u, symbol Device:C
- added C17, C18, C19, C20, C21, C22: 100n, symbol Device:C
- added C23, C24: 1u, symbol Device:C
- added FB2: 120R, symbol Device:FerriteBead
- added J2: USB_C_Receptacle_USB2.0_16P, Connector_USB:USB_C_Receptacle_GCT_USB4105-xx-A_16P_TopMnt_Horizontal, symbol Connector:USB_C_Receptacle_USB2.0_16P
- added R6: 5k1, symbol Device:R
- added U2: AP2112K-3.3, Package_TO_SOT_SMD:SOT-23-5, symbol Regulator_Linear:AP2112K-3.3
- added U3: USBLC6-2SC6, Package_TO_SOT_SMD:SOT-23-6, symbol Power_Protection:USBLC6-2SC6
- added U4: ICM-42688-P, User_Sensors:PQFN50P300X250X97-14N, symbol Sensor_Motion:ICM-42688-P
- C2, C3: value 100n -> 1u
- C5: value 100n -> 2.2u
- C6: value 100n -> 10n
Connections:
- net +3.3V: now also C4.2, C5.2, C16.1, C17.1, C18.1, C19.1, C20.1, C21.1, C22.1, C24.1, FB2.2, U2.5 (VOUT), U4.5 (VDDIO), U4.8 (VDD); no longer C1.1, C2.1, C4.1, C5.1
- net +3.3VA: now also C1.1, C2.1, FB2.1
- net +5V: now also C23.1, J2.A4 (VBUS), J2.A9 (VBUS), J2.B4 (VBUS), J2.B9 (VBUS), U2.1 (VIN), U2.3 (EN), U3.5 (VBUS)
- net D+: now also J2.A6 (D+), J2.B6 (D+), U3.1 (I/O1), U3.6 (I/O1)
- net D-: now also J2.A7 (D-), J2.B7 (D-), U3.3 (I/O2), U3.4 (I/O2)
- net GND: now also C4.1, C5.1, C16.2, C17.2, C18.2, C19.2, C20.2, C21.2, C22.2, C23.2, C24.2, J2.A1 (GND), J2.A12 (GND), J2.B1 (GND), J2.B12 (GND), J2.SH (SHIELD), R6.2, U2.2 (GND), U3.2 (GND), U4.6 (GND), U4.7 (RESV_7); no longer C4.2, C5.2
- net at R3.1: now also J2.B5 (CC2)
- new net: J2.A5 (CC1), R6.1
- no-connect marks 1 -> 2
Other:
- note added: "Analog Power Filtering"
- note added: "Digital Power Filtering"
- note added: "Power Conversion"
- note added: "USB ESD Protection"
- moved on the sheet: C11, C12, C13, C14, C15, J1, R1, R2, R3, SW1, TP4, TP5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

Commit message: Document flight controller design decisions
Parts:
- added C7: 100n, symbol Device:C_Small
- added C8: 100u 50V, symbol Device:C_Polarized
- added C9: 220u 25 V, symbol Device:C_Polarized
- added D1: 1N5825, symbol Device:D_Schottky
- added D4, D5: B5819W, symbol Device:D_Schottky
- added J3: ESC, symbol Connector_Generic:Conn_01x08
- added L2: 100u, symbol Device:L
- added R7: 10k, symbol Device:R_Small
- added R8: 15k, symbol Device:R_Small
- added R9: 100k, symbol Device:R_Small
- added U5: LM2596S-5, Package_TO_SOT_SMD:TO-263-5_TabPin3, symbol Regulator_Switching:LM2596S-5
Connections:
- net +3.3V: now also R7.1
- net +5V: now also D4.1 (K), D5.1 (K); no longer J2.A4 (VBUS), J2.A9 (VBUS), J2.B4 (VBUS), J2.B9 (VBUS), U3.5 (VBUS)
- net GND: now also C7.2, C8.2, C9.2, D1.2 (A), R8.2, U5.3 (GND), U5.5 (~{ON}/OFF)
- net IMU_MISO: now reaches U4.1 (AP_SDO/AP_AD0)
- net IMU_MISO: now also U1.30 (PA6)
- net IMU_SEL: now reaches U4.12 (AP_CS)
- net IMU_SEL: now also U1.34 (PB0), R7.2
- net IMU_CLK: now reaches U4.13 (AP_SCL/AP_SCLK)
- net IMU_CLK: now also U1.29 (PA5)
- net IMU_MOSI: now reaches U4.14 (AP_SDA/AP_SDIO/AP_SDI)
- net IMU_MOSI: now also U1.31 (PA7)
- net IMU_INTER: now reaches U4.4 (INT1/INT)
- net IMU_INTER: now also U1.32 (PC4)
- net BAT_SENSE: now reaches U1.15 (PC0)
- net BAT_SENSE: now also C7.1, R8.1, R9.2
- net MOTOR1: now reaches U1.22 (PA0)
- net MOTOR2: now reaches U1.23 (PA1)
- net MOTOR3: now reaches U1.24 (PA2)
- net MOTOR4: now reaches U1.25 (PA3)
- net RC_TX: now reaches U1.46 (PB10)
- net RC_RX: now reaches U1.47 (PB11)
- new net: D1.1 (K), L2.2, U5.2 (OUT)
- new net: C8.1, U5.1 (VIN)
- new net BAT_4S: R9.1
- new net BUCK_5V: C9.1, D4.2 (A), L2.1, U5.4 (FB)
- new net USB_VBUS: D5.2 (A), J2.A4 (VBUS), J2.A9 (VBUS), J2.B4 (VBUS), J2.B9 (VBUS), U3.5 (VBUS)
- no-connect marks 2 -> 6
Other:
- note added: "4SBAT to 5V Buck Converter"
- note added: "Power Conversion 5V -> 3V3"
- note removed: "Power Conversion"
- moved on the sheet: C4, C5, C6, U4

Commit message: Add V1 drone MCU prototype and project plan
Parts:
- added C24: 100n, symbol Device:C_Small
- added D1: B260A(LS), symbol Device:D_Schottky
- added D5: SMBJ20A, symbol Device:D_Zener
- added J4: RECIVER, symbol Connector_Generic:Conn_01x04
- added JP1: SolderJumper_2_Open, symbol Jumper:SolderJumper_2_Open
- added TP6: BAT_SENSE, symbol Connector:TestPoint
- R7: renamed from R8; value 15k -> 10k
- renumbered C16 to C1, C3 to C10, C8 to C12, C23 to C13, C24 to C14, C9 to C15, C14 to C16, C15 to C17, C7 to C18, C13 to C19, C17 to C2, C12 to C20, C4 to C21, C5 to C22, C6 to C23, C18 to C3, C19 to C4, C20 to C5, C21 to C6, C22 to C7, C1 to C8, C2 to C9, D1 to D2, D4 to D3, D5 to D4, FB2 to FB1, J3 to J1, J1 to J2, J2 to J3, L2 to L1, R4 to R3, R5 to R4, R9 to R5, R3 to R8, R7 to R9, TP5 to TP1, TP4 to TP2, TP6 to TP3, TP7 to TP4, TP8 to TP5, U5 to U1, U1 to U3, U3 to U4, U4 to U5, Y2 to Y1
Connections:
- net +5V: now also C24.1, J4.1 (Pin_1)
- net BAT_4S: now also J1.7 (Pin_7), D1.2 (A); no longer R5.1
- net BAT_SENSE: now also JP1.2 (B), TP6.1; no longer U3.15 (PC0)
- net GND: now also J1.8 (Pin_8), C24.2, D5.2 (A), J4.2 (Pin_2)
- net MOTOR1: now also J1.6 (Pin_6)
- net MOTOR2: now also J1.5 (Pin_5)
- net MOTOR3: now also J1.4 (Pin_4)
- net MOTOR4: now also J1.3 (Pin_3)
- net RC_RX: now also J4.3 (Pin_3)
- net RC_TX: now also J4.4 (Pin_4)
- net BUCK_IN: now reaches C12.1, U1.1 (VIN)
- net BUCK_IN: now also R5.1, D1.1 (K), D5.1 (K)
- new net ADC_BAT: JP1.1 (A), U3.15 (PC0)
Other:
- note added: "IMU"
- moved on the sheet: C10, C12, C13, C14, C15, C18, C19, C20, C21, C22, C23, C8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
